File: StarbieSchematic/StarbieSchematic.kicad_pcb (KiCad board)
At the start: 2 copper layers, 127 x 127 mm, 11 parts, among them J1 Conn_01x04_Pin, J2 Conn_01x08_Pin, SW1 SW_Push, SW2 SW_Push, U1 XIAO-ESP32-C3-SMD, U2 DHT11

Commit message: BOM and new footprints for starbie
Parts:
- added G***: LOGO, ImageConverter:nebula, F.Cu at (102.9, 100.3)
- added G***: LOGO, ImageConverter:star2, F.Cu at (204.5, 82.5)
- moved G*** 5.68 mm to (144.8, 137.2)
