File: StarbieSchematic/StarbieSchematic.kicad_sch (KiCad schematic)
At the start: 0 parts

Commit message: started building schematic
Parts:
- added SW1, SW2: SW_Push, symbol Switch:SW_Push
- added U1: XIAO-ESP32-C3-SMD, Seeed_Studio_XIAO_Series:XIAO-ESP32-C3-SMD, symbol Seeed_Studio_XIAO_Series:XIAO-ESP32-C3-SMD
Connections:
- new net +3.3V: U1.12 (3V3_OUT)
- new net +5V: U1.14 (VBUS)
- new net GND: SW1.2, SW2.2, U1.13 (GND), U1.18 (GND)
- new net GPIO2: SW1.1
- new net GPIO3: SW2.1

Commit message: Done with pcb
Parts:
- added J1: Conn_01x04_Pin, Imported Parts:Display_128x64_096_I2C, symbol Connector:Conn_01x04_Pin
- added J2: Conn_01x08_Pin, Connector_PinHeader_2.54mm:PinHeader_1x08_P2.54mm_Vertical, symbol Connector:Conn_01x08_Pin
- added R1: 10K, Resistor_THT:R_Axial_DIN0204_L3.6mm_D1.6mm_P7.62mm_Horizontal, symbol Device:R
- added U2: DHT11, Sensor:Aosong_DHT11_5.5x12.0_P2.54mm, symbol Sensor:DHT11
- SW1, SW2: footprint (none) -> Button_Switch_Keyboard:SW_Cherry_MX_1.00u_PCB
- U1: footprint Seeed_Studio_XIAO_Series:XIAO-ESP32-C3-SMD -> Imported Parts:XIAO-ESP32-C6-DIP
Connections:
- net +3.3V: now also J1.2 (Pin_2), J2.1 (Pin_1), R1.1, U2.1 (VDD)
- net GND: now also J1.1 (Pin_1), J2.2 (Pin_2), U2.4 (GND)
- net GPIO2: now also U1.3 (D2)
- net GPIO3: now also U1.4 (D3)
- net DHT11 DATA: now reaches U1.2 (D1)
- net DHT11 DATA: now also R1.2, U2.2 (DATA)
- net SCL: now reaches U1.5 (D4)
- net SCL: now also J1.3 (Pin_3), J2.3 (Pin_3)
- net SDA: now reaches U1.6 (D5)
- net SDA: now also J1.4 (Pin_4), J2.4 (Pin_4)
- no-connect marks 0 -> 13

Commit message: BOM and new footprints for starbie
Other:
- title: (none) -> Starbie Schematic
Changed lines of the file:
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@@
 	(generator_version "10.0")
 	(paper "A4")
+	(title_block
+		(title "Starbie Schematic")
+	)
 	(no_connect
 		(at 59.69 50.8)
